File: hardware/kicad/fan_controller.kicad_pcb (KiCad board)
At the start: 2 copper layers, 75 x 60 mm, 78 parts, among them J1 12V IN, J10 AIN2, J11 AIN3, J12 AIN4, J13 AIN5, J14 AIN6, J2 BluePill A, J3 BluePill B, J5 FAN1, J6 FAN2, J7 FAN3, J8 FAN4, J9 AIN1, Q1 BSS138, Q2 BSS138, Q3 BSS138, Q4 BSS138

Commit message: hw: clear DRC/ERC library and dangling-net warnings
Remove 4 dangling track stubs and 6 vestigial single-layer vias left
over from prior routing cleanup. Sync J1 (Mate-N-Lok) footprint
against its fanctl library copy by adding the missing attr/
remove_unused_layers flags, clearing the lib_footprint_mismatch
warning. Resync 68 standard-part footprints (R/C/L/Fuse/SOT-23/
PinHeader/PinSocket) against the now-installed KiCad system
libraries: swap stale multi-segment silk/fab/courtyard graphics for
the current library primitives, and fix oval-vs-circle pad shape
drift on PinHeader_1x03/PinSocket_1x20 (same pad size, cosmetic only).

DRC: 0 errors, 149 -> 66 warnings (remaining are silk_overlap/
silk_over_copper only). ERC: 81 -> 3 warnings (pre-existing
single-pin-label notices only). gen_kicad.py untouched.

Signed-off-by: Roman Skakun <rm.skakun@gmail.com>
Routing:
- net GND: track 359.0 -> 356.5 mm, vias 6 -> 5
- net +3V3: track 189.1 -> 188.1 mm, vias 7 -> 5
- net FAN4_PWM: vias 2 -> 0
- net FAN1_TACH: vias 4 -> 3
- net +3V3A: vias 8 -> 7
