File: hardware/kicad/fan_controller.kicad_pcb (KiCad board)
At the start: 2 copper layers, 81 x 78 mm, 115 parts, among them J1 12V IN, J10 AIN2, J11 AIN3, J12 AIN4, J13 AIN5, J14 AIN6, J2 BluePill A, J3 BluePill B, J5 FAN1, J6 FAN2, J7 FAN3, J8 FAN4, J9 AIN1, Q1 BSS138, Q10 BSS138, Q11 AO3401A, Q12 MMBT3906, Q13 BSS138, Q14 AO3401A, Q15 MMBT3906, Q16 BSS138, Q17 BSS138, Q18 BSS138, Q19 BSS138, Q2 BSS138, Q20 BSS138, Q3 BSS138, Q4 BSS138, Q5 AO3401A, Q6 MMBT3906, Q7 BSS138, Q8 AO3401A, Q9 MMBT3906

Commit message: PCB small corrections and rerouting
Signed-off-by: Roman Skakun <rm.skakun@gmail.com>
Parts:
- moved R45 2.24 mm to (64.3, 19.0)
- moved R47 0.96 mm to (59.5, 18.0), turned to 90 degrees
Routing:
- net AIN4: track 73.4 -> 76.8 mm
- net FAN4_TACH: track 62.1 -> 58.8 mm
- net GND: track 662.2 -> 659.0 mm
- net FAN4_DCEN: track 28.4 -> 30.9 mm
- net FAN3_TACH: track 78.6 -> 76.6 mm
- net V12_SENSE: track 51.6 -> 53.3 mm
- net VIN_12V: track 19.9 -> 18.4 mm
- net FAN2_TACH_IN: track 35.9 -> 37.4 mm
- net Net-(Q17-D): track 80.6 -> 79.3 mm
- net FAN1_DCEN: track 59.4 -> 60.7 mm
- net FAN4_PWM: track 80.0 -> 80.9 mm
- net FAN2_DCEN: track 53.1 -> 54.1 mm
