File: hardware/kicad/fan_controller.kicad_sch (KiCad schematic)
At the start: 124 parts, among them J1 12V IN, J10 AIN2, J11 AIN3, J12 AIN4, J13 AIN5, J14 AIN6, J2 SWD, J3 USB micro-B, J4 USB int, J5 FAN1, J6 FAN2, J7 FAN3, J8 FAN4, J9 AIN1, Q1 IRLML6402, Q10 IRLML6402, Q11 BSS138, Q12 BSS138, Q2 BSS138, Q3 BSS138, Q4 IRLML6402, Q5 BSS138, Q6 BSS138, Q7 IRLML6402, Q8 BSS138, Q9 BSS138, U1 AMS1117-3.3, U2 STM32F103C8T6, U3 USBLC6-2SC6, Y1 8MHz

Commit message: hw: replace discontinued P-FET, protect LDO, fuse each fan
- AO3401A (-30 V) replaces the discontinued IRLML6402. The 30 V rating
  also covers the SMBJ13A's 21.5 V clamp.
- 47 R feed and 13 V zener hold the AMS1117 input below its 15 V limit
  during rail surges.
- Tantalum output capacitor for AMS1117 stability.
- 1.1 A PTC per fan channel, so one shorted fan does not trip F1.
- Six test pads: +12V, +3V3, GND, NRST, FAN1_PWM, FAN1_TACH.

Signed-off-by: Roman Skakun <rm.skakun@gmail.com>
Parts:
- added D18: BAT54S, Package_TO_SOT_SMD:SOT-23, symbol fanctl:BAT54S
- added F2, F3, F4, F5: 1.1A, Fuse:Fuse_1812_4532Metric, symbol fanctl:Polyfuse
- added R51: 1k, Resistor_SMD:R_0603_1608Metric, symbol fanctl:R
- added TP1: +12V, TestPoint:TestPoint_Pad_D1.5mm, symbol fanctl:TestPoint
- added TP2: +3V3, TestPoint:TestPoint_Pad_D1.5mm, symbol fanctl:TestPoint
- added TP3: GND, TestPoint:TestPoint_Pad_D1.5mm, symbol fanctl:TestPoint
- added TP4: NRST, TestPoint:TestPoint_Pad_D1.5mm, symbol fanctl:TestPoint
- added TP5: FAN1_PWM, TestPoint:TestPoint_Pad_D1.5mm, symbol fanctl:TestPoint
- added TP6: FAN1_TACH, TestPoint:TestPoint_Pad_D1.5mm, symbol fanctl:TestPoint
- C4: footprint Capacitor_SMD:C_1206_3216Metric -> Capacitor_Tantalum_SMD:CP_EIA-3528-21_Kemet-B; symbol fanctl:C -> fanctl:C_Pol; MPN (none) -> KEMET T491B226K010AT
- D10, D6, D8: value BZT52C10 -> SS14; footprint Diode_SMD:D_SOD-123 -> Diode_SMD:D_SMA; symbol fanctl:D_Zener -> fanctl:D_Schottky; MPN Diodes Inc BZT52C10-7-F -> SS14
- D11, D5, D7, D9: value SS14 -> BZT52C10; footprint Diode_SMD:D_SMA -> Diode_SMD:D_SOD-123; symbol fanctl:D_Schottky -> fanctl:D_Zener; MPN SS14 -> Diodes Inc BZT52C10-7-F
- D12: value BAT54S -> SS14; footprint Package_TO_SOT_SMD:SOT-23 -> Diode_SMD:D_SMA; symbol fanctl:BAT54S -> fanctl:D_Schottky; MPN Nexperia BAT54S,215 -> SS14
- D3: value green -> BZT52C13; footprint LED_SMD:LED_0603_1608Metric -> Diode_SMD:D_SOD-123; symbol fanctl:LED -> fanctl:D_Zener; MPN (none) -> Diodes Inc BZT52C13-7-F
- D4: value BZT52C10 -> green; footprint Diode_SMD:D_SOD-123 -> LED_SMD:LED_0603_1608Metric; symbol fanctl:D_Zener -> fanctl:LED; MPN Diodes Inc BZT52C10-7-F -> (none)
- Q1, Q10, Q4, Q7: value IRLML6402 -> AO3401A; MPN Infineon IRLML6402TRPBF -> Alpha & Omega AO3401A
- R1: value 47k -> 47; footprint Resistor_SMD:R_0603_1608Metric -> Resistor_SMD:R_1206_3216Metric
- R10, R18, R26, R34: value 10k -> 100
- R11, R19, R27, R35: value 100 -> 10k
- R12, R20, R28, R36: value 100k -> 100
- R13, R21, R29, R37: value 10k -> 100k
- R14, R22, R30, R38, R40, R42, R44, R46, R48, R5, R50: value 1k -> 10k
- R15, R23, R31: value 4k7 -> 1k
- R17, R25, R33, R9: value 100 -> 4k7
- R2: value 10k -> 47k
- R39, R41, R43, R45, R47, R49: value 10k -> 1k
- R6: value 1k5 -> 1k
- R7: value 4k7 -> 1k5
Connections:
- net +12V: now also D11.1 (K), D5.1 (K), D7.1 (K), D9.1 (K), R16.1, R2.1, R24.1, R32.1, R8.1, TP1.1; no longer D10.1 (K), D2.2 (A2), D4.1 (K), D6.1 (K), D8.1 (K), R15.1, R23.1, R31.1, R7.1
- net +3V3: now also R11.2, R14.2, R19.2, R22.2, R27.2, R30.2, R35.2, R38.2, R6.1, R7.2, TP2.1; no longer R10.2, R13.2, R18.2, R21.2, R26.2, R29.2, R34.2, R37.2, R5.1, R6.2
- net +3V3A: now also R40.2, R42.2, R44.2, R46.2, R48.2, R50.2, D18.2 (K2); no longer D12.2 (K2), R39.2, R41.2, R43.2, R45.2, R47.2, R49.2
- net AIN1: now also D13.3 (K1A2), R41.2; no longer D12.3 (K1A2), R40.2
- net AIN1_IN: now also R41.1; no longer R39.1
- net AIN2: now also D14.3 (K1A2), R43.2; no longer D13.3 (K1A2), R42.2
- net AIN2_IN: now also R43.1; no longer R41.1
- net AIN3: now also D15.3 (K1A2), R45.2; no longer D14.3 (K1A2), R44.2
- net AIN3_IN: now also R45.1; no longer R43.1
- net AIN4: now also D16.3 (K1A2), R47.2; no longer D15.3 (K1A2), R46.2
- net AIN4_IN: now also R47.1; no longer R45.1
- net AIN5: now also D17.3 (K1A2), R49.2; no longer D16.3 (K1A2), R48.2
- net AIN5_IN: now also R49.1; no longer R47.1
- net AIN6: now also D18.3 (K1A2), R51.2; no longer D17.3 (K1A2), R50.2
- net AIN6_IN: now also R51.1; no longer R49.1
- net BOOT0: now also R4.1; no longer R3.1
- net BOOT1: now also R5.1; no longer R4.1
- net FAN1_12V: now also D6.1 (K), F2.2; no longer D5.1 (K), Q1.3 (D)
- net FAN1_DRV: now also R9.2; no longer R8.2
- net FAN1_GATE: now also D5.2 (A), R8.2, R9.1; no longer D4.2 (A), R7.2, R8.1
- net FAN1_PWM: now also R12.1, TP5.1; no longer R11.1
- net FAN1_PWM_G: now also R12.2, R13.1; no longer R11.2, R12.1
- net FAN1_PWR: now also R10.1; no longer R9.1
- net FAN1_PWR_G: now also R10.2, R11.1; no longer R10.1, R9.2
- net FAN1_TACH: now also R15.2, TP6.1; no longer R14.2
- net FAN1_TACH_IN: now also R15.1; no longer R13.1
- net FAN2_12V: now also D8.1 (K), F3.2; no longer D7.1 (K), Q4.3 (D)
- net FAN2_DRV: now also R17.2; no longer R16.2
- net FAN2_GATE: now also D7.2 (A), R16.2, R17.1; no longer D6.2 (A), R15.2, R16.1
- net FAN2_PWM: now also R20.1; no longer R19.1
- net FAN2_PWM_G: now also R20.2, R21.1; no longer R19.2, R20.1
- net FAN2_PWR: now also R18.1; no longer R17.1
- net FAN2_PWR_G: now also R18.2, R19.1; no longer R17.2, R18.1
- net FAN2_TACH: now also R23.2; no longer R22.2
- net FAN2_TACH_IN: now also R23.1; no longer R21.1
- net FAN3_12V: now also D10.1 (K), F4.2; no longer D9.1 (K), Q7.3 (D)
- net FAN3_DRV: now also R25.2; no longer R24.2
- net FAN3_GATE: now also D9.2 (A), R24.2, R25.1; no longer D8.2 (A), R23.2, R24.1
- net FAN3_PWM: now also R28.1; no longer R27.1
- net FAN3_PWM_G: now also R28.2, R29.1; no longer R27.2, R28.1
- net FAN3_PWR: now also R26.1; no longer R25.1
- net FAN3_PWR_G: now also R26.2, R27.1; no longer R25.2, R26.1
- net FAN3_TACH: now also R31.2; no longer R30.2
- net FAN3_TACH_IN: now also R31.1; no longer R29.1
- net FAN4_12V: now also D12.1 (K), F5.2; no longer D11.1 (K), Q10.3 (D)
- net FAN4_DRV: now also R33.2; no longer R32.2
- net FAN4_GATE: now also D11.2 (A), R32.2, R33.1; no longer D10.2 (A), R31.2, R32.1
- net FAN4_PWM: now also R36.1; no longer R35.1
- net FAN4_PWM_G: now also R36.2, R37.1; no longer R35.2, R36.1
- net FAN4_PWR: now also R34.1; no longer R33.1
- net FAN4_PWR_G: now also R34.2, R35.1; no longer R33.2, R34.1
- net FAN4_TACH: now also R39.2; no longer R38.2
- net FAN4_TACH_IN: now also R39.1; no longer R37.1
- net GND: now also D10.2 (A), D12.2 (A), D3.2 (A), D6.2 (A), D8.2 (A), R13.2, R21.2, R29.2, R37.2, R5.2, D18.1 (A1), TP3.1; no longer D11.2 (A), D12.1 (A1), D5.2 (A), D7.2 (A), D9.2 (A), R12.2, R2.2, R20.2, R28.2, R36.2
- net LED_A: now also D4.2 (A), R6.2; no longer D3.2 (A), R5.2
- net LED_K: now also D4.1 (K); no longer D3.1 (K)
- net NRST: now also TP4.1
- net USB_DP: now also R7.1; no longer R6.1
- net V12_SENSE: now also R2.2, R3.1; no longer R1.2, R2.1
- net VREG_IN: now also D3.1 (K)
- new net FAN1_SW_12V: F2.1, Q1.3 (D)
- new net FAN2_SW_12V: F3.1, Q4.3 (D)
- new net FAN3_SW_12V: F4.1, Q7.3 (D)
- new net FAN4_SW_12V: F5.1, Q10.3 (D)
- new net V12_LDO: D2.2 (A2), R1.2
Other:
- note added: "Test points"
- moved on the sheet: C16, C17, C18, C19, C3, C5, C6, C7, D10, D11, D13, D14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

Commit message: hw: Blue Pill carrier, first placement and 3D model
The board is now a carrier for an STM32F103C8T6 Blue Pill module in two
1x20 sockets. The module brings the MCU, crystal, 3.3 V regulator, LED,
reset, BOOT jumpers, SWD and micro-B USB, so those parts are removed.
An AMS1117-5.0 feeds the module's 5V pin through an SS14, which stops
USB VBUS from back-feeding the regulator. R4 (DNP) corrects modules
whose D+ pull-up is 10k. Header pinout follows the DeepBlueMbedded
Blue Pill diagram.

place_pcb.py places every footprint by block (placed, not routed),
checks overlaps, board edges and mounting holes, and exports
fan_controller.step and .glb. The STEP models are committed under
hardware/kicad/3dmodels/ and referenced through ${KIPRJMOD}, so KiCad
uses them without the 3D library installed. pcb_top.png heads the
README.

Signed-off-by: Roman Skakun <rm.skakun@gmail.com>
Parts:
- removed C18, C19: 1n, Capacitor_SMD:C_0603_1608Metric, symbol fanctl:C
- removed C20, C21, C22, C23, C24, C25: 100n, Capacitor_SMD:C_0603_1608Metric, symbol fanctl:C
- removed D18: BAT54S, Package_TO_SOT_SMD:SOT-23, symbol fanctl:BAT54S
- removed R49, R51: 1k, Resistor_SMD:R_0603_1608Metric, symbol fanctl:R
- removed R50: 10k, Resistor_SMD:R_0603_1608Metric, symbol fanctl:R
- removed U3: USBLC6-2SC6, Package_TO_SOT_SMD:SOT-23-6, symbol fanctl:USBLC6-2SC6
- removed Y1: 8MHz, Crystal:Crystal_SMD_3225-4Pin_3.2x2.5mm, symbol fanctl:Crystal_GND24
- C10, C11, C8, C9: value 100n -> 1n
- C12: value 4u7 -> 100n; footprint Capacitor_SMD:C_1206_3216Metric -> Capacitor_SMD:C_0603_1608Metric
- C13, C14: value 27p -> 100n
- C16, C17: value 1n -> 100n
- D10, D6, D8: value SS14 -> BZT52C10; footprint Diode_SMD:D_SMA -> Diode_SMD:D_SOD-123; symbol fanctl:D_Schottky -> fanctl:D_Zener; MPN SS14 -> Diodes Inc BZT52C10-7-F
- D11, D5, D7, D9: value BZT52C10 -> SS14; footprint Diode_SMD:D_SOD-123 -> Diode_SMD:D_SMA; symbol fanctl:D_Zener -> fanctl:D_Schottky; MPN Diodes Inc BZT52C10-7-F -> SS14
- D12: value SS14 -> BAT54S; footprint Diode_SMD:D_SMA -> Package_TO_SOT_SMD:SOT-23; symbol fanctl:D_Schottky -> fanctl:BAT54S; MPN SS14 -> Nexperia BAT54S,215
- D2: value BAT54C -> BZT52C13; footprint Package_TO_SOT_SMD:SOT-23 -> Diode_SMD:D_SOD-123; symbol fanctl:BAT54C -> fanctl:D_Zener; MPN Nexperia BAT54C,215 -> Diodes Inc BZT52C13-7-F
- D3: value BZT52C13 -> SS14; footprint Diode_SMD:D_SOD-123 -> Diode_SMD:D_SMA; symbol fanctl:D_Zener -> fanctl:D_Schottky; MPN Diodes Inc BZT52C13-7-F -> SS14
- D4: value green -> BZT52C10; footprint LED_SMD:LED_0603_1608Metric -> Diode_SMD:D_SOD-123; symbol fanctl:LED -> fanctl:D_Zener; MPN (none) -> Diodes Inc BZT52C10-7-F
- J2: value SWD -> BluePill A; footprint Connector_PinHeader_2.54mm:PinHeader_1x05_P2.54mm_Vertical -> Connector_PinSocket_2.54mm:PinSocket_1x20_P2.54mm_Vertical; symbol fanctl:Conn_01x05 -> fanctl:BluePill_A
- J3: value USB micro-B -> BluePill B; footprint Connector_USB:USB_Micro-B_Molex-105017-0001 -> Connector_PinSocket_2.54mm:PinSocket_1x20_P2.54mm_Vertical; symbol fanctl:USB_B_Micro -> fanctl:BluePill_B; MPN Molex 105017-0001 -> (none)
- R10, R18, R26, R34: value 100 -> 100k
- R12, R20, R28, R36: value 100 -> 1k
- R13, R21, R29: value 100k -> 4k7
- R14, R22, R30, R5: value 10k -> 4k7
- R15, R23, R31: value 1k -> 100
- R16, R24, R32, R8: value 4k7 -> 10k
- R17, R25, R33, R9: value 4k7 -> 100
- R37: value 100k -> 10k
- R38, R40, R42, R44, R46, R48: value 10k -> 1k
- R39, R41, R43, R45, R47: value 1k -> 10k
- R4: value 10k -> 1k8; now not fitted
- R6: value 1k -> 4k7
- R7: value 1k5 -> 100
- U1: value AMS1117-3.3 -> AMS1117-5.0; symbol fanctl:AMS1117-3.3 -> fanctl:AMS1117; MPN AMS1117-3.3 -> AMS1117-5.0
- U2: value STM32F103C8T6 -> USBLC6-2SC6; footprint Package_QFP:LQFP-48_7x7mm_P0.5mm -> Package_TO_SOT_SMD:SOT-23-6; symbol fanctl:STM32F103C8Tx -> fanctl:USBLC6-2SC6; MPN STMicroelectronics STM32F103C8T6 -> STMicroelectronics USBLC6-2SC6
Connections:
- net +12V: now also D10.1 (K), D4.1 (K), D6.1 (K), D8.1 (K), R13.1, R21.1, R29.1, R5.1; no longer D11.1 (K), D5.1 (K), D7.1 (K), D9.1 (K), R16.1, R24.1, R32.1, R8.1
- net +3V3: now also J2.3 (3V3), J3.20 (3V3), R16.2, R24.2, R32.2, R4.2, R8.2; no longer C10.1, C11.1, C12.1, C4.1 (+), C8.1, C9.1, J2.1, R14.2, R22.2, R30.2, R38.2, R6.1, R7.2, U1.2 (VO), U2.1 (VBAT), U2.24 (VDD), U2.36 (VDD), U2.48 (VDD)
- net +3V3A: now also D12.2 (K2), R37.2, R39.2, R41.2, R43.2, R45.2, R47.2; no longer R40.2, R42.2, R44.2, R46.2, R48.2, U2.9 (VDDA)
- net AIN1: now also C12.1, D12.3 (K1A2), J2.16 (PA0), R38.2; no longer D13.3 (K1A2), R41.2, U2.10 (PA0)
- net AIN1_IN: now also R37.1, R38.1; no longer R40.1, R41.1
- net AIN2: now also C13.1, D13.3 (K1A2), J2.15 (PA1), R40.2; no longer D14.3 (K1A2), R43.2, U2.11 (PA1)
- net AIN2_IN: now also R39.1, R40.1; no longer R42.1, R43.1
- net AIN3: now also C14.1, D14.3 (K1A2), J2.14 (PA2), R42.2; no longer D15.3 (K1A2), R45.2, U2.12 (PA2)
- net AIN3_IN: now also R41.1, R42.1; no longer R44.1, R45.1
- net AIN4: now also C15.1, D15.3 (K1A2), J2.13 (PA3), R44.2; no longer D16.3 (K1A2), R47.2, U2.13 (PA3)
- net AIN4_IN: now also R43.1, R44.1; no longer R46.1, R47.1
- net AIN5: now also C16.1, D16.3 (K1A2), J2.12 (PA4), R46.2; no longer D17.3 (K1A2), U2.14 (PA4)
- net AIN5_IN: now also R45.1, R46.1; no longer R48.1
- net AIN6: now also C17.1, D17.3 (K1A2), J2.11 (PA5), R48.2; no longer U2.15 (PA5)
- net AIN6_IN: now also R47.1, R48.1
- net FAN1_12V: now also D5.1 (K); no longer D6.1 (K)
- net FAN1_DRV: now also R6.2; no longer R9.2
- net FAN1_GATE: now also D4.2 (A), R5.2, R6.1; no longer D5.2 (A), R8.2, R9.1
- net FAN1_PWM: now also J3.14 (PB6), R9.1; no longer R12.1, U2.42 (PB6)
- net FAN1_PWM_G: now also R10.1, R9.2; no longer R12.2, R13.1
- net FAN1_PWR: now also J3.10 (PA15), R7.1; no longer R10.1, U2.38 (PA15)
- net FAN1_PWR_G: now also R7.2, R8.1; no longer R10.2, R11.1
- net FAN1_TACH: now also C8.1, J3.1 (PB12), R12.2; no longer C16.1, R15.2, U2.25 (PB12)
- net FAN1_TACH_IN: now also R11.1, R12.1; no longer R14.1, R15.1
- net FAN2_12V: now also D7.1 (K); no longer D8.1 (K)
- net FAN2_DRV: now also R14.2; no longer R17.2
- net FAN2_GATE: now also D6.2 (A), R13.2, R14.1; no longer D7.2 (A), R16.2, R17.1
- net FAN2_PWM: now also J3.15 (PB7), R17.1; no longer R20.1, U2.43 (PB7)
- net FAN2_PWM_G: now also R17.2, R18.1; no longer R20.2, R21.1
- net FAN2_PWR: now also J3.11 (PB3), R15.1; no longer R18.1, U2.39 (PB3)
- net FAN2_PWR_G: now also R15.2, R16.1; no longer R18.2, R19.1
- net FAN2_TACH: now also C9.1, J3.2 (PB13), R20.2; no longer C17.1, R23.2, U2.26 (PB13)
- net FAN2_TACH_IN: now also R19.1, R20.1; no longer R22.1, R23.1
- net FAN3_12V: now also D9.1 (K); no longer D10.1 (K)
- net FAN3_DRV: now also R22.2; no longer R25.2
- net FAN3_GATE: now also D8.2 (A), R21.2, R22.1; no longer D9.2 (A), R24.2, R25.1
- net FAN3_PWM: now also J3.16 (PB8), R25.1; no longer R28.1, U2.45 (PB8)
- net FAN3_PWM_G: now also R25.2, R26.1; no longer R28.2, R29.1
- net FAN3_PWR: now also J2.6 (PB10), R23.1; no longer R26.1, U2.21 (PB10)
- net FAN3_PWR_G: now also R23.2, R24.1; no longer R26.2, R27.1
- net FAN3_TACH: now also C10.1, J3.3 (PB14), R28.2; no longer R31.2, U2.27 (PB14)
- net FAN3_TACH_IN: now also R27.1, R28.1; no longer R30.1, R31.1
- net FAN4_12V: now also D11.1 (K); no longer D12.1 (K)
- net FAN4_DRV: now also R30.2; no longer R33.2
- net FAN4_GATE: now also D10.2 (A), R29.2, R30.1; no longer D11.2 (A), R32.2, R33.1
- net FAN4_PWM: now also J3.17 (PB9), R33.1; no longer R36.1, U2.46 (PB9)
- net FAN4_PWM_G: now also R33.2, R34.1; no longer R36.2, R37.1
- net FAN4_PWR: now also J2.5 (PB11), R31.1; no longer R34.1, U2.22 (PB11)
- net FAN4_PWR_G: now also R31.2, R32.1; no longer R34.2, R35.1
- net FAN4_TACH: now also C11.1, J3.4 (PB15), R36.2; no longer R39.2, U2.28 (PB15)
- net FAN4_TACH_IN: now also R35.1, R36.1; no longer R38.1, R39.1
- net GND: now also D11.2 (A), D12.1 (A1), D2.2 (A), D5.2 (A), D7.2 (A), D9.2 (A), J2.1 (GND), J2.2 (GND), J3.19 (GND), R10.2, R18.2, R26.2, R34.2, U2.2 (GND); no longer D10.2 (A), D12.2 (A), D3.2 (A), D6.2 (A), D8.2 (A), J2.3, J3.5 (GND), J3.6 (Shield), R13.2, R21.2, R29.2, R37.2, R4.2, R5.2, U2.23 (VSS), U2.35 (VSS), U2.47 (VSS), U2.8 (VSSA)
- net NRST: now also J2.4 (NRST); no longer C15.1, J2.5, U2.7 (NRST)
- net USB_DM: now also J3.8 (PA11), U2.3 (IO2), U2.4 (IO2); no longer J3.2 (D-), U2.32 (PA11)
- net USB_DP: now also J3.9 (PA12), R4.1, U2.1 (IO1), U2.6 (IO1); no longer J3.3 (D+), R7.1, U2.33 (PA12)
- net V12_SENSE: now also J2.8 (PB0); no longer U2.18 (PB0)
- net VREG_IN: now also D2.1 (K), R1.2; no longer D2.3 (K), D3.1 (K)
- removed net BOOT0: R4.1, U2.44 (BOOT0)
- removed net BOOT1: R5.1, U2.20 (PB2)
- removed net LED_A: D4.2 (A), R6.2
- removed net LED_K: D4.1 (K), U2.2 (PC13)
- net OSC_IN renamed +5V
- net +5V: now also D3.1 (K), J3.18 (5V), J4.1; no longer C13.1
- removed net OSC_OUT: C14.1, U2.6 (PD1-OSC_OUT)
- removed net SWCLK: J2.2, U2.37 (PA14)
- removed net SWDIO: J2.4, U2.34 (PA13)
- removed net V12_LDO: D2.2 (A2), R1.2
- removed net VBUS: D2.1 (A1), J3.1 (VBUS), J4.1
- new net +5V_REG: C4.1 (+), D3.2 (A), U1.2 (VO)
- no-connect marks 11 -> 12
Other:
- moved on the sheet: C10, C11, C12, C13, C14, C15, C16, C17, C3, C4, C5, C6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

Commit message: hw: power Blue Pill from USB, feed fans straight from 12 V
The Blue Pill now runs from USB only, so the AMS1117-5.0 and its
protection (47 R, 13 V zener, tantalum, SS14 OR diode) are removed.

Fan pin 2 connects to +12 V through its 1.1 A PTC. The high-side
P-FET, its gate network, level shifter and freewheel diode are gone
from every channel. Fans now run at 100 % whenever the module is
unpowered, held in reset or missing, because the PWM buffer releases
the line. Before, unplugging USB would have switched every fan off.
3-pin fans and the hard stop at 0 % are no longer supported.

Firmware 2.0 drops TIM2 and the mode command; get no longer prints
mode=. fanctl.py drops its mode subcommand.

The board shrinks from 100 x 80 mm to 75 x 60 mm and from 122 to 84
parts. Board size now lives in gen_kicad.py and is shared with
place_pcb.py. Placement, STEP, GLB and renders are regenerated, and
unused 3D models are removed. README replaces the safety prose with
a failure-case table.

Signed-off-by: Roman Skakun <rm.skakun@gmail.com>
Parts:
- removed C16, C17: 100n, Capacitor_SMD:C_0603_1608Metric, symbol fanctl:C
- removed D10, D8: BZT52C10, Diode_SMD:D_SOD-123, symbol fanctl:D_Zener
- removed D11, D9: SS14, Diode_SMD:D_SMA, symbol fanctl:D_Schottky
- removed D12, D13, D14, D15, D16, D17: BAT54S, Package_TO_SOT_SMD:SOT-23, symbol fanctl:BAT54S
- removed Q10, Q7: AO3401A, Package_TO_SOT_SMD:SOT-23, symbol fanctl:Q_PMOS_GSD
- removed Q11, Q12, Q5, Q6, Q8, Q9: BSS138, Package_TO_SOT_SMD:SOT-23, symbol fanctl:Q_NMOS_GSD
- removed R32, R35, R37, R39, R41, R43, R45, R47: 10k, Resistor_SMD:R_0603_1608Metric, symbol fanctl:R
- removed R33: 100, Resistor_SMD:R_0603_1608Metric, symbol fanctl:R
- removed R34: 100k, Resistor_SMD:R_0603_1608Metric, symbol fanctl:R
- removed R36, R38, R40, R42, R44, R46, R48: 1k, Resistor_SMD:R_0603_1608Metric, symbol fanctl:R
- removed U2: USBLC6-2SC6, Package_TO_SOT_SMD:SOT-23-6, symbol fanctl:USBLC6-2SC6
- C10, C11: value 1n -> 100n
- C3: value 10u 25V -> 1u; footprint Capacitor_SMD:C_1206_3216Metric -> Capacitor_SMD:C_0603_1608Metric
- C4: value 22u 10V -> 10n; footprint Capacitor_Tantalum_SMD:CP_EIA-3528-21_Kemet-B -> Capacitor_SMD:C_0603_1608Metric; symbol fanctl:C_Pol -> fanctl:C; MPN KEMET T491B226K010AT -> (none)
- C5: value 1u -> 100n
- C6: value 10n -> 1n
- C7: value 100n -> 1n
- D2: value BZT52C13 -> BAT54S; footprint Diode_SMD:D_SOD-123 -> Package_TO_SOT_SMD:SOT-23; symbol fanctl:D_Zener -> fanctl:BAT54S; MPN Diodes Inc BZT52C13-7-F -> Nexperia BAT54S,215
- D3, D5, D7: value SS14 -> BAT54S; footprint Diode_SMD:D_SMA -> Package_TO_SOT_SMD:SOT-23; symbol fanctl:D_Schottky -> fanctl:BAT54S; MPN SS14 -> Nexperia BAT54S,215
- D4, D6: value BZT52C10 -> BAT54S; footprint Diode_SMD:D_SOD-123 -> Package_TO_SOT_SMD:SOT-23; symbol fanctl:D_Zener -> fanctl:BAT54S; MPN Diodes Inc BZT52C10-7-F -> Nexperia BAT54S,215
- Q1, Q4: value AO3401A -> BSS138; symbol fanctl:Q_PMOS_GSD -> fanctl:Q_NMOS_GSD; MPN Alpha & Omega AO3401A -> onsemi BSS138
- R1: value 47 -> 47k; footprint Resistor_SMD:R_1206_3216Metric -> Resistor_SMD:R_0603_1608Metric
- R10, R18, R26: value 100k -> 10k
- R11, R19, R27: value 10k -> 1k
- R12: value 1k -> 100
- R13, R5: value 4k7 -> 100k
- R14, R22, R30, R6: value 4k7 -> 10k
- R15, R23, R25, R31, R7: value 100 -> 1k
- R16, R8: value 10k -> 100
- R17, R9: value 100 -> 100k
- R2: value 47k -> 10k
- R20, R28: value 1k -> 10k
- R21, R29: value 4k7 -> 1k
- R3: value 10k -> 1k8; now not fitted
- R4: value 1k8 -> 100; now fitted
- U1: value AMS1117-5.0 -> USBLC6-2SC6; footprint Package_TO_SOT_SMD:SOT-223-3_TabPin2 -> Package_TO_SOT_SMD:SOT-23-6; symbol fanctl:AMS1117 -> fanctl:USBLC6-2SC6; MPN AMS1117-5.0 -> STMicroelectronics USBLC6-2SC6
Connections:
- net FAN2_DRV is gone; now on net +3V3: R14.2
- net FAN3_DRV is gone; now on net +3V3A: R22.2
- net FAN3_SW_12V is gone; now on net +12V: F4.1
- net FAN4_DRV is gone; now on net +3V3A: R30.2
- net FAN4_PWR_G is gone; now on net AIN6: R31.2
- net FAN4_SW_12V is gone; now on net +12V: F5.1
- net +12V: now also F2.1, F3.1; no longer D4.1 (K), D6.1 (K), Q1.2 (S), Q4.2 (S), R13.1, R2.1, R21.1, R29.1, R5.1
- net +3V3: now also R10.2, R18.2, R3.2, R6.2; no longer R11.2, R16.2, R19.2, R24.2, R27.2, R4.2, R8.2
- net +3V3A: now also C3.1, C4.1, D2.2 (K2), D3.2 (K2), D4.2 (K2), D5.2 (K2), D6.2 (K2), D7.2 (K2), R20.2, R24.2, R26.2, R28.2; no longer C5.1, C6.1
- net +5V: now also U1.5 (VBUS); no longer D3.1 (K)
- net AIN1: now also C10.1, D2.3 (K1A2), R21.2; no longer C12.1
- net AIN1_IN: now also R20.1, R21.1
- net AIN2: now also C11.1, D3.3 (K1A2), R23.2; no longer C13.1
- net AIN2_IN: now also R22.1, R23.1
- net AIN3: now also C12.1, D4.3 (K1A2), R25.2; no longer C14.1
- net AIN3_IN: now also R24.1, R25.1
- net AIN4: now also C13.1, D5.3 (K1A2), R27.2; no longer C15.1
- net AIN4_IN: now also R26.1, R27.1
- net AIN5: now also C14.1, D6.3 (K1A2), R29.2
- net AIN5_IN: now also R28.1, R29.1
- net AIN6: now also C15.1, D7.3 (K1A2)
- net AIN6_IN: now also R30.1, R31.1
- net FAN1_12V: no longer D5.1 (K)
- net FAN1_PWM: now also R4.1; no longer R9.1
- net FAN1_PWM_G: now also Q1.1 (G), R4.2, R5.1; no longer Q3.1 (G), R10.1, R9.2
- net FAN1_PWM_OUT: now also Q1.3 (D); no longer Q3.3 (D)
- net FAN1_TACH: now also C6.1, R7.2; no longer C8.1, R12.2
- net FAN1_TACH_IN: now also R6.1, R7.1; no longer R11.1, R12.1
- net FAN2_12V: no longer D7.1 (K)
- net FAN2_PWM: now also R8.1; no longer R17.1
- net FAN2_PWM_G: now also Q2.1 (G), R8.2, R9.1; no longer R17.2, R18.1
- net FAN2_PWM_OUT: now also Q2.3 (D)
- net FAN2_TACH: now also C7.1, R11.2; no longer C9.1, R20.2
- net FAN2_TACH_IN: now also R10.1, R11.1; no longer R19.1, R20.1
- net FAN3_PWM: now also R12.1; no longer R25.1
- net FAN3_PWM_G: now also Q3.1 (G), R12.2, R13.1; no longer R25.2, R26.1
- net FAN3_PWM_OUT: now also Q3.3 (D)
- net FAN3_TACH: now also C8.1, R15.2; no longer C10.1, R28.2
- net FAN3_TACH_IN: now also R14.1, R15.1; no longer R27.1, R28.1
- net FAN4_PWM: now also R16.1
- net FAN4_PWM_G: now also Q4.1 (G), R16.2, R17.1
- net FAN4_PWM_OUT: now also Q4.3 (D)
- net FAN4_TACH: now also C9.1, R19.2; no longer C11.1
- net FAN4_TACH_IN: now also R18.1, R19.1
- net GND: now also D2.1 (A1), D3.1 (A1), D4.1 (A1), D5.1 (A1), D6.1 (A1), D7.1 (A1), Q1.2 (S), Q4.2 (S), R13.2, R17.2, R2.2, R5.2, R9.2, U1.2 (GND); no longer D2.2 (A), D5.2 (A), D7.2 (A), R10.2, R18.2, R26.2, R3.2, U1.1 (GND)
- net USB_DM: now also U1.3 (IO2), U1.4 (IO2)
- net USB_DP: now also R3.1, U1.1 (IO1), U1.6 (IO1); no longer R4.1
- net V12_SENSE: now also C5.1, R1.2, R2.1; no longer C7.1, R2.2, R3.1
- removed net +5V_REG: C4.1 (+), D3.2 (A), U1.2 (VO)
- removed net FAN1_DRV: Q2.3 (D), R6.2
- removed net FAN1_GATE: D4.2 (A), Q1.1 (G), R5.2, R6.1
- net FAN1_PWR: no longer names the net of J3.10 (PA15)
- net FAN1_PWR: no longer R7.1
- removed net FAN1_PWR_G: Q2.1 (G), R7.2, R8.1
- removed net FAN1_SW_12V: F2.1, Q1.3 (D)
- removed net FAN2_GATE: D6.2 (A), Q4.1 (G), R13.2, R14.1
- net FAN2_PWR: no longer names the net of J3.11 (PB3)
- net FAN2_PWR: no longer R15.1
- removed net FAN2_PWR_G: R15.2, R16.1
- removed net FAN2_SW_12V: F3.1, Q4.3 (D)
- removed net FAN3_GATE: R21.2, R22.1
- net FAN3_PWR: no longer names the net of J2.6 (PB10)
- net FAN3_PWR: no longer R23.1
- removed net FAN3_PWR_G: R23.2, R24.1
- removed net FAN4_GATE: R29.2, R30.1
- net FAN4_PWR: no longer names the net of J2.5 (PB11)
- net FAN4_PWR: no longer R31.1
- removed net VREG_IN: C3.1, D2.1 (K), R1.2, U1.3 (VI)
- no-connect marks 12 -> 16
Other:
- moved on the sheet: C10, C11, C12, C13, C14, C15, C3, C5, C6, C7, C8, C9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
