File: hardware/kicad/fan_controller.kicad_sch (KiCad schematic)
At the start: 75 parts, among them J1 12V IN, J10 AIN2, J11 AIN3, J12 AIN4, J13 AIN5, J14 AIN6, J2 BluePill A, J3 BluePill B, J5 FAN1, J6 FAN2, J7 FAN3, J8 FAN4, J9 AIN1, Q1 BSS138, Q2 BSS138, Q3 BSS138, Q4 BSS138

Commit message: rename project to Fanny, drop gen_kicad.py/place_pcb.py generator scripts
Title: "Fanny - a versatile USB PWM fan controller" (README, schematic
and PCB title blocks).

KiCad files are now hand-maintained directly and are the source of
truth; place_pcb.py depended on gen_kicad.py's PARTS table and had no
purpose without it. Updated README's KiCad project section, folder
tree, and 3dmodels/README.md accordingly, and the schematic's stale
"generated by" comment.

Signed-off-by: Roman Skakun <rm.skakun@gmail.com>
Other:
- title: STM32F103 PWM fan controller -> Fanny - versatile USB PWM fan controller
Changed lines of the file:
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@@
 	(paper "A1")
 	(title_block
-		(title "STM32F103 PWM fan controller")
+		(title "Fanny - versatile USB PWM fan controller")
 		(rev "1.0")
-		(comment 1 "Generated by hardware/tools/gen_kicad.py - edit the script, not this file")
-	)
+		)
 	(text "Analog inputs"
 		(exclude_from_sim no)

Commit message: DC mode support
Signed-off-by: Roman Skakun <rm.skakun@gmail.com>
Parts:
- added D10, D11, D8, D9: SS34, Diode_SMD:D_SMA, symbol fanctl:D
- added JP1, JP2, JP3, JP4: 0, Resistor_SMD:R_1206_3216Metric, symbol fanctl:R
- added Q10, Q13, Q16, Q17, Q18, Q19, Q20, Q7: BSS138, Package_TO_SOT_SMD:SOT-23, symbol fanctl:Q_NMOS_GSD
- added Q11, Q14, Q5, Q8: AO3401A, Package_TO_SOT_SMD:SOT-23, symbol Transistor_FET:Q_PMOS_GSD
- added Q12, Q15, Q6, Q9: MMBT3906, Package_TO_SOT_SMD:SOT-23, symbol Transistor_BJT:MMBT3906
- added R32, R35, R38, R41: 2.2k, Resistor_SMD:R_0603_1608Metric, symbol fanctl:R
- added R33, R36, R39, R42, R44, R45, R46, R47: 10k, Resistor_SMD:R_0603_1608Metric, symbol fanctl:R
- added R34, R37, R40, R43: 4.7k, Resistor_SMD:R_0603_1608Metric, symbol fanctl:R
Connections:
- net FAN1_12V: now also D8.1 (K), JP1.2, Q5.3 (D); no longer F2.2
- net FAN1_PWM_G: no longer R5.1
- net FAN1_TACH: no longer C6.1
- net FAN2_12V: now also D9.1 (K), JP2.2, Q8.3 (D); no longer F3.2
- net FAN2_PWM_G: now also Q10.1 (G); no longer R9.1
- net FAN2_TACH: no longer C7.1
- net FAN2_TACH_IN: no longer R11.1
- net FAN3_12V: now also D10.1 (K), JP3.2, Q11.3 (D); no longer F4.2
- net FAN3_PWM_G: now also Q13.1 (G); no longer R13.1
- net FAN3_TACH: no longer C8.1
- net FAN3_TACH_IN: no longer R15.1
- net FAN4_12V: now also D11.1 (K), JP4.2, Q14.3 (D); no longer F5.2
- net FAN4_PWM_G: now also Q16.1 (G); no longer R17.1
- net FAN4_TACH: no longer C9.1
- net GND: now also D11.2 (A), D8.2 (A), D9.2 (A), Q17.2 (S), Q18.2 (S), Q19.2 (S), Q20.2 (S), R35.2, R38.2, R41.2, R44.2, R45.2, R46.2, R47.2; no longer C1.2 (-), C10.2, C11.2, C12.2, C13.2, C14.2, C15.2, C2.2, C3.2, C4.2, C5.2, D1.2 (A), D2.1 (A1), D3.1 (A1), D4.1 (A1), D5.1 (A1), D7.1 (A1), J1.3, J1.4, J11.3, J12.3, J14.3, J2.1 (GND), J2.2 (GND), J3.19 (GND), J9.3, R2.2
- net FAN1_DCEN: now reaches J2.10 (PA6)
- net FAN1_DCEN: now also Q17.1 (G), R44.1
- net FAN4_DCEN: now reaches J2.7 (PB1)
- net FAN4_DCEN: now also Q20.1 (G), R47.1
- net FAN2_DCEN: now reaches J2.9 (PA7)
- net FAN2_DCEN: now also Q18.1 (G), R45.1
- net FAN3_DCEN: now reaches J3.5 (PA8)
- net FAN3_DCEN: now also Q19.1 (G), R46.1
- new net: Q13.2 (S), Q19.3 (D)
- new net: Q17.3 (D), Q7.2 (S)
- new net: Q16.2 (S), Q20.3 (D)
- new net: Q10.2 (S), Q18.3 (D)
- new net +12V_F1: F2.2, JP1.1, Q5.2 (S), Q6.2 (E), R33.2
- new net +12V_F2: F3.2, JP2.1, Q8.2 (S), Q9.2 (E), R36.2
- new net +12V_F3: F4.2, JP3.1, Q11.2 (S), Q12.2 (E), R39.2
- new net +12V_F4: F5.2, JP4.1, Q14.2 (S), Q15.2 (E), R42.2
- new net FAN1_BASE: Q6.1 (B), R33.1, R34.1
- new net FAN1_GATE: Q5.1 (G), Q6.3 (C), R32.1
- new net FAN1_RB_INV: Q7.3 (D), R34.2
- new net FAN2_BASE: Q9.1 (B), R36.1, R37.1
- new net FAN2_GATE: Q8.1 (G), Q9.3 (C), R35.1
- new net FAN2_RB_INV: Q10.3 (D), R37.2
- new net FAN3_BASE: Q12.1 (B), R39.1, R40.1
- new net FAN3_GATE: Q11.1 (G), Q12.3 (C), R38.1
- new net FAN3_RB_INV: Q13.3 (D), R40.2
- new net FAN4_BASE: Q15.1 (B), R42.1, R43.1
- new net FAN4_GATE: Q14.1 (G), Q15.3 (C), R41.1
- new net FAN4_RB_INV: Q16.3 (D), R43.2
- no-connect marks 16 -> 12
Other:
- note removed: "Test points"
- moved on the sheet: J2, J3, J5, J6, J7, J8

Commit message: hw: fix schematic connectivity errors and sync PCB to new nets
Convert local labels to global labels so net names stop getting a
sheet-path prefix (/+12V vs +12V) on PCB sync. Add missing junction
markers at four T-tapped gate-drive/tach points that touch a crossing
wire's body but weren't bonded to it, and missing GND symbols on the
channel-1 gate-bias resistor, channel-3 flyback diode, and the AIN
clamp/filter network. Resolve a duplicate #PWR101 annotation. Sync the
PCB from the schematic now that nets match cleanly (ERC 57->17
violations, 41->13 errors).

Signed-off-by: Roman Skakun <rm.skakun@gmail.com>
Connections:
- net FAN1_PWM_G: now also Q7.1 (G), R5.1
- net FAN1_TACH: now also C6.1
- net FAN2_PWM_G: now also R9.1
- net FAN2_TACH: now also C7.1
- net FAN2_TACH_IN: now also R11.1
- net FAN3_PWM_G: now also R13.1
- net FAN3_TACH: now also C8.1
- net FAN3_TACH_IN: now also R15.1
- net FAN4_PWM_G: now also R17.1
- net FAN4_TACH: now also C9.1
- net GND: now also C10.2, C11.2, C12.2, C13.2, C14.2, C15.2, D10.2 (A), D2.1 (A1), D3.1 (A1), D4.1 (A1), D5.1 (A1), D7.1 (A1), J11.3, J12.3, J14.3, J9.3, R32.2

Commit message: hw: clean up motor-switch duplicate footprints and dead-net shorts
Remove stray duplicate Q17/Q18/Q19/Q20 (Q_en) and R44-R47 (R_dcen)
footprints left over from PCB sync, and delete the leftover copper on
the resulting dead Net-(Qn-...) nets that was shorting the live
Q_inv/Q_en cascode nets (Net-(Q13-S), Net-(Q16-S), Net-(Q17-D)).
Reconnect J2 pin1/pin2 to GND in the schematic (found floating, no
wire or power symbol). Align the 4 board-perimeter bolt holes into a
clean rectangle (one corner was 0.1mm off). DRC shorting_items for
this feature's nets cleared; remaining DRC errors are pre-existing and
out of scope.

Signed-off-by: Roman Skakun <rm.skakun@gmail.com>
Connections:
- net FAN4_TACH_IN is gone; now on net FAN4_PWM_G: J8.3 (Tach), R18.1, R19.1
- net AIN1: now also J2.13 (PA3); no longer J2.16 (PA0)
- net AIN2: now also J2.14 (PA2); no longer J2.15 (PA1)
- net AIN3: now also J2.15 (PA1); no longer J2.14 (PA2)
- net AIN4: now also J2.16 (PA0); no longer J2.13 (PA3)
- net GND: now also J2.1 (GND), J2.2 (GND)
Other:
- moved on the sheet: J7, R39, R40
